File: tweezer-tips/tweezer-tips.kicad_pcb (KiCad board)
At the start: 2 copper layers, 140.5 x 10 mm, 5 parts, among them J1 TIP, J2 TO_AMP, J3 GND

Commit message: Revision 2
Parts:
- added R2: 220, Resistor_SMD:R_0603_1608Metric, F.Cu at (148.0, 100.0)
- C1: value 0.5pF -> 1.0pF
- J2: footprint oscilloscope-probes:SIMPLE_PAD -> TestPoint:TestPoint_THTPad_D1.0mm_Drill0.5mm
- R1: value 9.1M -> 9.53M
- moved J3 36.8 mm to (226.2, 101.4)
- moved J2 9.60 mm to (228.9, 100.0)
- moved C1 6.80 mm to (151.0, 99.2)
- moved R1 6.80 mm to (151.0, 100.8)
Connections:
- C1 pad 1: /TIP -> Net-(C1-Pad1)
- R1 pad 2: /TIP -> Net-(C1-Pad1)
Routing:
- net GND: track 181.6 -> 136.6 mm, vias 8 -> 6
- net /TIP: track 23.6 -> 14.8 mm
- net Net-(C1-Pad1): track 0.00 -> 2.89 mm
Other:
- board size 140.5 x 10 mm -> 130 x 10 mm
- board text added: "1:1 1 MΩ"
- board text added: "1:10 10 MΩ"
- board text added: "Enclosure front edge"

Commit message: Revision 3
Parts:
- added C2: N/A, Capacitor_SMD:C_0603_1608Metric, F.Cu at (153.6, 100.8)
- added E1: SPARK_GAP, oscilloscope-probes:PCB_SPARK_GAP, F.Cu at (143.4, 100.0)
- added E2: SPARK_GAP, oscilloscope-probes:PCB_SPARK_GAP, F.Cu at (161.0, 100.0)
Routing:
- net /AMP: track 81.9 -> 78.6 mm
- net GND: track 136.6 -> 136.7 mm, vias 6 -> 8
Other:
- outline, holes or cut-outs redrawn
- net class Default: clearance 0.2 -> 0.14
- rule trace_clearance: 0.2 -> 0.14
- board text added: "1:2 1 MΩ"
- board text added: "1:20 10 MΩ"
- board text added: "CAT I 100 Vpk"
- board text added: "Main pcb front edge"
- board text removed: "1:1 1 MΩ"
- board text removed: "1:10 10 MΩ"
- board text removed: "Enclosure front edge"
