File: tweezer-tips/tweezer-tips.sch (KiCad schematic (older format))
At the start: 5 parts, among them J1 TIP, J2 TO_AMP, J3 GND

Commit message: Revision 2
Parts:
- added R2: 220, Resistor_SMD:R_0603_1608Metric, symbol Device:R
- C1: value 0.5pF -> 1.0pF
- J2: footprint oscilloscope-probes:SIMPLE_PAD -> TestPoint:TestPoint_THTPad_D1.0mm_Drill0.5mm
- R1: value 9.1M -> 9.53M
Connections:
- net TIP: now also R2.2; no longer C1.1, R1.2
- new net: C1.1, R1.2, R2.1
Changed lines of the file:
@@
 F 0 "J2" H 6878 3676 50  0000 L CNN
 F 1 "TO_AMP" H 6878 3585 50  0000 L CNN
-F 2 "oscilloscope-probes:SIMPLE_PAD" H 6850 3650 50  0001 C CNN
+F 2 "TestPoint:TestPoint_THTPad_D1.0mm_Drill0.5mm" H 6850 3650 50  0001 C CNN
 F 3 "~" H 6850 3650 50  0001 C CNN
 	1    6850 3650
@@
 P 4950 3500
 F 0 "R1" V 4743 3500 50  0000 C CNN
-F 1 "9.1M" V 4834 3500 50  0000 C CNN
+F 1 "9.53M" V 4834 3500 50  0000 C CNN
 F 2 "Resistor_SMD:R_0603_1608Metric" V 4880 3500 50  0001 C CNN
 F 3 "~" H 4950 3500 50  0001 C CNN
@@
 P 4950 3800
 F 0 "C1" V 4790 3800 50  0000 C CNN
-F 1 "0.5pF" V 4699 3800 50  0000 C CNN
+F 1 "1.0pF" V 4699 3800 50  0000 C CNN
 F 2 "Capacitor_SMD:C_0603_1608Metric" H 4988 3650 50  0001 C CNN
 F 3 "~" H 4950 3800 50  0001 C CNN
@@
 $EndComp
 Wire Wire Line
-	3550 3650 4750 3650
-Wire Wire Line
-	4750 3650 4750 3500
-Wire Wire Line
 	4750 3500 4800 3500
 Wire Wire Line
-	4750 3650 4750 3800
-Wire Wire Line
 	4750 3800 4800 3800
-Connection ~ 4750 3650
 Wire Wire Line
 	5100 3800 5200 3800
@@
 Text Label 5700 3650 0    50   ~ 0
 AMP
+Wire Wire Line
+	4750 3500 4750 3650
+$Comp
+L Device:R R2
+U 1 1 609904A1
+P 4600 3650
+F 0 "R2" V 4393 3650 50  0000 C CNN
+F 1 "220" V 4484 3650 50  0000 C CNN
+F 2 "Resistor_SMD:R_0603_1608Metric" V 4530 3650 50  0001 C CNN
+F 3 "~" H 4600 3650 50  0001 C CNN
+	1    4600 3650
+	0    1    1    0
+$EndComp
+Connection ~ 4750 3650
+Wire Wire Line
+	4750 3650 4750 3800
+Wire Wire Line
+	4450 3650 3550 3650
 $EndSCHEMATC

Commit message: Revision 3
Parts:
- added C2: N/A, Capacitor_SMD:C_0603_1608Metric, symbol Device:C
- added E1, E?: SPARK_GAP, oscilloscope-probes:PCB_SPARK_GAP, symbol Device:SPARK_GAP
Connections:
- net AMP: now also C2.1, E?.1
- net GND: now also C2.2, E1.2, E?.2
- net TIP: now also E1.1
Changed lines of the file:
@@
 	5200 3800 5200 3650
 Wire Wire Line
-	5200 3650 6650 3650
+	5200 3650 5600 3650
 Wire Wire Line
 	5100 3500 5200 3500
@@
 L power:GND #PWR01
 U 1 1 5FFCB4EE
-P 5800 4400
-F 0 "#PWR01" H 5800 4150 50  0001 C CNN
-F 1 "GND" H 5805 4227 50  0000 C CNN
-F 2 "" H 5800 4400 50  0001 C CNN
-F 3 "" H 5800 4400 50  0001 C CNN
-	1    5800 4400
+P 5600 4400
+F 0 "#PWR01" H 5600 4150 50  0001 C CNN
+F 1 "GND" H 5605 4227 50  0000 C CNN
+F 2 "" H 5600 4400 50  0001 C CNN
+F 3 "" H 5600 4400 50  0001 C CNN
+	1    5600 4400
 	1    0    0    -1
 $EndComp
@@
 $EndComp
 Wire Wire Line
-	6650 4300 5800 4300
+	6650 4300 6150 4300
 Wire Wire Line
-	5800 4300 5800 4400
-Text Label 3950 3650 0    50   ~ 0
+	5600 4300 5600 4400
+Text Label 3750 3650 0    50   ~ 0
 TIP
 Text Label 5700 3650 0    50   ~ 0
@@
 	4750 3650 4750 3800
 Wire Wire Line
-	4450 3650 3550 3650
+	4450 3650 4000 3650
+$Comp
+L Device:C C2
+U 1 1 60B603A2
+P 5600 4000
+F 0 "C2" H 5715 4046 50  0000 L CNN
+F 1 "N/A" H 5715 3955 50  0000 L CNN
+F 2 "Capacitor_SMD:C_0603_1608Metric" H 5638 3850 50  0001 C CNN
+F 3 "~" H 5600 4000 50  0001 C CNN
+	1    5600 4000
+	1    0    0    -1
+$EndComp
+Connection ~ 5600 3650
+Wire Wire Line
+	5600 3650 6150 3650
+Wire Wire Line
+	5600 3850 5600 3650
+Wire Wire Line
+	5600 4150 5600 4300
+Connection ~ 5600 4300
+$Comp
+L Device:SPARK_GAP E1
+U 1 1 60B619A9
+P 4000 4000
+F 0 "E1" V 3954 4053 50  0000 L CNN
+F 1 "SPARK_GAP" V 4045 4053 50  0000 L CNN
+F 2 "oscilloscope-probes:PCB_SPARK_GAP" H 4000 3930 50  0001 C CNN
+F 3 "~" V 4000 4000 50  0001 C CNN
+	1    4000 4000
+	0    1    1    0
+$EndComp
+Wire Wire Line
+	4000 4300 5600 4300
+Wire Wire Line
+	4000 4300 4000 4200
+Wire Wire Line
+	4000 3800 4000 3650
+Connection ~ 4000 3650
+Wire Wire Line
+	4000 3650 3550 3650
+$Comp
+L Device:SPARK_GAP E?
+U 1 1 60B63DD8
+P 6150 4000
+F 0 "E?" V 6104 4053 50  0000 L CNN
+F 1 "SPARK_GAP" V 6195 4053 50  0000 L CNN
+F 2 "oscilloscope-probes:PCB_SPARK_GAP" H 6150 3930 50  0001 C CNN
+F 3 "~" V 6150 4000 50  0001 C CNN
+	1    6150 4000
+	0    1    1    0
+$EndComp
+Wire Wire Line
+	6150 4200 6150 4300
+Connection ~ 6150 4300
+Wire Wire Line
+	6150 4300 5600 4300
+Wire Wire Line
+	6150 3800 6150 3650
+Connection ~ 6150 3650
+Wire Wire Line
+	6150 3650 6650 3650
 $EndSCHEMATC

Commit message: BOM updates
Parts:
- gave numbers to parts that had none: 1
Changed lines of the file:
@@
 	4000 3650 3550 3650
 $Comp
-L Device:SPARK_GAP E?
+L Device:SPARK_GAP E2
 U 1 1 60B63DD8
 P 6150 4000
-F 0 "E?" V 6104 4053 50  0000 L CNN
+F 0 "E2" V 6104 4053 50  0000 L CNN
 F 1 "SPARK_GAP" V 6195 4053 50  0000 L CNN
 F 2 "oscilloscope-probes:PCB_SPARK_GAP" H 6150 3930 50  0001 C CNN
