File: cable_to_banana/cable_to_banana.sch (KiCad schematic (older format))
At the start: 15 parts, among them J1 Banana, J2 Coax center, J3 Coax shield

Commit message: BOM updates
Parts:
- C1, C2, C3, C4, C5: value 10pF 2kV -> 10pF; Mfg (none) -> KEMET; Mfg Part No (none) -> C1206C100FGGAC7800; Notes (none) -> NP0, 1%, >= 600V
- C6: value N/A -> 360pF; Mfg (none) -> KEMET; Mfg Part No (none) -> C0603C361G5GAC7867; Notes (none) -> NP0, 2%
- J1: footprint Connector_PinHeader_2.54mm:PinHeader_1x01_P2.54mm_Horizontal -> oscilloscope-probes:SIMPLE_PAD; Mfg (none) -> CalTech; Mfg Part No (none) -> CT3204
- R1, R2, R3, R4, R5: Mfg (none) -> Bourns; Mfg Part No (none) -> CHV1206-FX-1005ELF; Notes (none) -> 1%, >= 600V
Other:
- note added: "C6 must be chosen according to cable capacitance.\nThe total capacitance of cable plus the 20 pF nominal amplifier\ncapacitance must be 400 pF."
Changed lines of the file:
@@
 F 0 "J1" H 2808 2981 50  0000 C CNN
 F 1 "Banana" H 2808 2890 50  0000 C CNN
-F 2 "Connector_PinHeader_2.54mm:PinHeader_1x01_P2.54mm_Horizontal" H 2700 2800 50  0001 C CNN
+F 2 "oscilloscope-probes:SIMPLE_PAD" H 2700 2800 50  0001 C CNN
 F 3 "~" H 2700 2800 50  0001 C CNN
+F 4 "CalTech" H 2700 2800 50  0001 C CNN "Mfg"
+F 5 "CT3204" H 2700 2800 50  0001 C CNN "Mfg Part No"
 	1    2700 2800
 	1    0    0    -1
@@
 F 2 "oscilloscope-probes:Minimal1206" V 3280 2800 50  0001 C CNN
 F 3 "~" H 3350 2800 50  0001 C CNN
+F 4 "Bourns" H 3350 2800 50  0001 C CNN "Mfg"
+F 5 "CHV1206-FX-1005ELF" H 3350 2800 50  0001 C CNN "Mfg Part No"
+F 6 "1%, >= 600V" H 3350 2800 50  0001 C CNN "Notes"
 	1    3350 2800
 	0    1    1    0
@@
 F 2 "oscilloscope-probes:Minimal1206" V 3780 2800 50  0001 C CNN
 F 3 "~" H 3850 2800 50  0001 C CNN
+F 4 "Bourns" H 3850 2800 50  0001 C CNN "Mfg"
+F 5 "CHV1206-FX-1005ELF" H 3850 2800 50  0001 C CNN "Mfg Part No"
+F 6 "1%, >= 600V" H 3850 2800 50  0001 C CNN "Notes"
 	1    3850 2800
 	0    1    1    0
@@
 P 6250 2950
 F 0 "C6" H 6365 2904 50  0000 L CNN
-F 1 "N/A" H 6365 2995 50  0000 L CNN
+F 1 "360pF" H 6365 2995 50  0000 L CNN
 F 2 "Capacitor_SMD:C_0603_1608Metric" H 6288 2800 50  0001 C CNN
 F 3 "~" H 6250 2950 50  0001 C CNN
+F 4 "C0603C361G5GAC7867" H 6250 2950 50  0001 C CNN "Mfg Part No"
+F 5 "KEMET" H 6250 2950 50  0001 C CNN "Mfg"
+F 6 "NP0, 2%" H 6250 2950 50  0001 C CNN "Notes"
 	1    6250 2950
 	-1   0    0    1
@@
 P 3350 3100
 F 0 "C1" V 3510 3100 50  0000 C CNN
-F 1 "10pF 2kV" V 3601 3100 50  0000 C CNN
+F 1 "10pF" V 3601 3100 50  0000 C CNN
 F 2 "oscilloscope-probes:Minimal1206" H 3388 2950 50  0001 C CNN
 F 3 "~" H 3350 3100 50  0001 C CNN
+F 4 "NP0, 1%, >= 600V" H 3350 3100 50  0001 C CNN "Notes"
+F 5 "KEMET" H 3350 3100 50  0001 C CNN "Mfg"
+F 6 "C1206C100FGGAC7800" H 3350 3100 50  0001 C CNN "Mfg Part No"
 	1    3350 3100
 	0    1    1    0
@@
 P 3850 3100
 F 0 "C2" V 4010 3100 50  0000 C CNN
-F 1 "10pF 2kV" V 4101 3100 50  0000 C CNN
+F 1 "10pF" V 4101 3100 50  0000 C CNN
 F 2 "oscilloscope-probes:Minimal1206" H 3888 2950 50  0001 C CNN
 F 3 "~" H 3850 3100 50  0001 C CNN
+F 4 "NP0, 1%, >= 600V" H 3850 3100 50  0001 C CNN "Notes"
+F 5 "KEMET" H 3850 3100 50  0001 C CNN "Mfg"
+F 6 "C1206C100FGGAC7800" H 3850 3100 50  0001 C CNN "Mfg Part No"
 	1    3850 3100
 	0    1    1    0
@@
 F 2 "oscilloscope-probes:Minimal1206" V 4280 2800 50  0001 C CNN
 F 3 "~" H 4350 2800 50  0001 C CNN
+F 4 "Bourns" H 4350 2800 50  0001 C CNN "Mfg"
+F 5 "CHV1206-FX-1005ELF" H 4350 2800 50  0001 C CNN "Mfg Part No"
+F 6 "1%, >= 600V" H 4350 2800 50  0001 C CNN "Notes"
 	1    4350 2800
 	0    1    1    0
@@
 F 2 "oscilloscope-probes:Minimal1206" V 4780 2800 50  0001 C CNN
 F 3 "~" H 4850 2800 50  0001 C CNN
+F 4 "Bourns" H 4850 2800 50  0001 C CNN "Mfg"
+F 5 "CHV1206-FX-1005ELF" H 4850 2800 50  0001 C CNN "Mfg Part No"
+F 6 "1%, >= 600V" H 4850 2800 50  0001 C CNN "Notes"
 	1    4850 2800
 	0    1    1    0
@@
 P 4350 3100
 F 0 "C3" V 4510 3100 50  0000 C CNN
-F 1 "10pF 2kV" V 4601 3100 50  0000 C CNN
+F 1 "10pF" V 4601 3100 50  0000 C CNN
 F 2 "oscilloscope-probes:Minimal1206" H 4388 2950 50  0001 C CNN
 F 3 "~" H 4350 3100 50  0001 C CNN
+F 4 "NP0, 1%, >= 600V" H 4350 3100 50  0001 C CNN "Notes"
+F 5 "KEMET" H 4350 3100 50  0001 C CNN "Mfg"
+F 6 "C1206C100FGGAC7800" H 4350 3100 50  0001 C CNN "Mfg Part No"
 	1    4350 3100
 	0    1    1    0
@@
 P 4850 3100
 F 0 "C4" V 5010 3100 50  0000 C CNN
-F 1 "10pF 2kV" V 5101 3100 50  0000 C CNN
+F 1 "10pF" V 5101 3100 50  0000 C CNN
 F 2 "oscilloscope-probes:Minimal1206" H 4888 2950 50  0001 C CNN
 F 3 "~" H 4850 3100 50  0001 C CNN
+F 4 "NP0, 1%, >= 600V" H 4850 3100 50  0001 C CNN "Notes"
+F 5 "KEMET" H 4850 3100 50  0001 C CNN "Mfg"
+F 6 "C1206C100FGGAC7800" H 4850 3100 50  0001 C CNN "Mfg Part No"
 	1    4850 3100
 	0    1    1    0
@@
 F 2 "oscilloscope-probes:Minimal1206" V 5280 2800 50  0001 C CNN
 F 3 "~" H 5350 2800 50  0001 C CNN
+F 4 "Bourns" H 5350 2800 50  0001 C CNN "Mfg"
+F 5 "CHV1206-FX-1005ELF" H 5350 2800 50  0001 C CNN "Mfg Part No"
+F 6 "1%, >= 600V" H 5350 2800 50  0001 C CNN "Notes"
 	1    5350 2800
 	0    1    1    0
@@
 P 5350 3100
 F 0 "C5" V 5510 3100 50  0000 C CNN
-F 1 "10pF 2kV" V 5601 3100 50  0000 C CNN
+F 1 "10pF" V 5601 3100 50  0000 C CNN
 F 2 "oscilloscope-probes:Minimal1206" H 5388 2950 50  0001 C CNN
 F 3 "~" H 5350 3100 50  0001 C CNN
+F 4 "NP0, 1%, >= 600V" H 5350 3100 50  0001 C CNN "Notes"
+F 5 "KEMET" H 5350 3100 50  0001 C CNN "Mfg"
+F 6 "C1206C100FGGAC7800" H 5350 3100 50  0001 C CNN "Mfg Part No"
 	1    5350 3100
 	0    1    1    0
@@
 Wire Wire Line
 	7150 3100 6550 3100
+Text Notes 6050 4100 0    50   ~ 0
+C6 must be chosen according to cable capacitance.\nThe total capacitance of cable plus the 20 pF nominal amplifier\ncapacitance must be 400 pF.
 $EndSCHEMATC
