File: accessories/cable_to_banana/cable_to_banana.kicad_pcb (KiCad board)
At the start: 2 copper layers, 19 x 6 mm, 15 parts, among them J1 Banana, J2 Coax center, J3 Coax shield

Commit message: Revision 4
Parts:
- removed the C1 at (121.1, 106.8)
- removed the C2 at (124.5, 106.8)
- removed the C3 at (127.9, 106.8)
- removed the C4 at (131.3, 106.8)
- removed the C6 at (137.2, 109.3)
- removed the J1 at (120.9, 108.0)
- removed the J2 at (133.0, 108.0)
- removed the J3 at (136.3, 108.0)
- removed the R1 at (121.1, 109.2)
- removed the R2 at (124.5, 109.2)
- removed the R3 at (127.9, 109.2)
- removed the R4 at (131.3, 109.2)
- removed the R5 at (134.7, 109.2)
- removed the R6 at (137.2, 106.7)
- added C1: 10pF, oscilloscope-probes:Minimal1206, F.Cu at (59.5, 170.7)
- added C1: 10pF, oscilloscope-probes:Minimal1206, F.Cu at (82.0, 148.8)
- added C1: 10pF, oscilloscope-probes:Minimal1206, F.Cu at (59.5, 130.7)
- added C1: 10pF, oscilloscope-probes:Minimal1206, F.Cu at (59.5, 160.7)
- added C1: 10pF, oscilloscope-probes:Minimal1206, F.Cu at (59.5, 140.7)
- added C1: 10pF, oscilloscope-probes:Minimal1206, F.Cu at (59.5, 150.7)
- added C1: 10pF, oscilloscope-probes:Minimal1206, F.Cu at (82.0, 128.8)
- added C1: 10pF, oscilloscope-probes:Minimal1206, F.Cu at (82.0, 138.8)
- added C1: 10pF, oscilloscope-probes:Minimal1206, F.Cu at (82.0, 168.8)
- added C1: 10pF, oscilloscope-probes:Minimal1206, F.Cu at (82.0, 158.8)
- added C2: 10pF, oscilloscope-probes:Minimal1206, F.Cu at (56.1, 130.7)
- added C2: 10pF, oscilloscope-probes:Minimal1206, F.Cu at (85.4, 148.8)
- added C2: 10pF, oscilloscope-probes:Minimal1206, F.Cu at (56.1, 160.7)
- added C2: 10pF, oscilloscope-probes:Minimal1206, F.Cu at (56.1, 140.7)
- added C2: 10pF, oscilloscope-probes:Minimal1206, F.Cu at (56.1, 170.7)
- added C2: 10pF, oscilloscope-probes:Minimal1206, F.Cu at (56.1, 150.7)
- added C2: 10pF, oscilloscope-probes:Minimal1206, F.Cu at (85.4, 128.8)
- added C2: 10pF, oscilloscope-probes:Minimal1206, F.Cu at (85.4, 138.8)
- added C2: 10pF, oscilloscope-probes:Minimal1206, F.Cu at (85.4, 168.8)
- added C2: 10pF, oscilloscope-probes:Minimal1206, F.Cu at (85.4, 158.8)
- added C3: 10pF, oscilloscope-probes:Minimal1206, F.Cu at (52.7, 128.5)
- added C3: 10pF, oscilloscope-probes:Minimal1206, F.Cu at (88.8, 151.0)
- added C3: 10pF, oscilloscope-probes:Minimal1206, F.Cu at (52.7, 168.5)
- added C3: 10pF, oscilloscope-probes:Minimal1206, F.Cu at (52.7, 158.5)
- added C3: 10pF, oscilloscope-probes:Minimal1206, F.Cu at (52.7, 138.5)
- added C3: 10pF, oscilloscope-probes:Minimal1206, F.Cu at (52.7, 148.5)
- added C3: 10pF, oscilloscope-probes:Minimal1206, F.Cu at (88.8, 131.0)
- added C3: 10pF, oscilloscope-probes:Minimal1206, F.Cu at (88.8, 141.0)
- added C3: 10pF, oscilloscope-probes:Minimal1206, F.Cu at (88.8, 171.0)
- added C3: 10pF, oscilloscope-probes:Minimal1206, F.Cu at (88.8, 161.0)
- added C4: 10pF, oscilloscope-probes:Minimal1206, F.Cu at (49.3, 128.5)
- added C4: 10pF, oscilloscope-probes:Minimal1206, F.Cu at (92.2, 151.0)
- added C4: 10pF, oscilloscope-probes:Minimal1206, F.Cu at (49.3, 158.5)
- added C4: 10pF, oscilloscope-probes:Minimal1206, F.Cu at (49.3, 138.5)
- added C4: 10pF, oscilloscope-probes:Minimal1206, F.Cu at (49.3, 168.5)
- added C4: 10pF, oscilloscope-probes:Minimal1206, F.Cu at (49.3, 148.5)
- added C4: 10pF, oscilloscope-probes:Minimal1206, F.Cu at (92.2, 131.0)
- added C4: 10pF, oscilloscope-probes:Minimal1206, F.Cu at (92.2, 141.0)
- added C4: 10pF, oscilloscope-probes:Minimal1206, F.Cu at (92.2, 171.0)
- added C4: 10pF, oscilloscope-probes:Minimal1206, F.Cu at (92.2, 161.0)
- added C5: 10pF, oscilloscope-probes:Minimal1206, F.Cu at (45.9, 168.5)
- added C5: 10pF, oscilloscope-probes:Minimal1206, F.Cu at (45.9, 138.5)
- added C5: 10pF, oscilloscope-probes:Minimal1206, F.Cu at (45.9, 128.5)
- added C5: 10pF, oscilloscope-probes:Minimal1206, F.Cu at (45.9, 158.5)
- added C5: 10pF, oscilloscope-probes:Minimal1206, F.Cu at (45.9, 148.5)
- added C5: 10pF, oscilloscope-probes:Minimal1206, F.Cu at (95.6, 131.0)
- added C5: 10pF, oscilloscope-probes:Minimal1206, F.Cu at (95.6, 141.0)
- added C5: 10pF, oscilloscope-probes:Minimal1206, F.Cu at (95.6, 171.0)
- added C5: 10pF, oscilloscope-probes:Minimal1206, F.Cu at (95.6, 161.0)
- added C6: 360pF, Capacitor_SMD:C_0603_1608Metric, F.Cu at (43.0, 140.2)
- added C6: 360pF, Capacitor_SMD:C_0603_1608Metric, F.Cu at (98.5, 149.3)
- added C6: 360pF, Capacitor_SMD:C_0603_1608Metric, F.Cu at (43.0, 130.2)
- added C6: 360pF, Capacitor_SMD:C_0603_1608Metric, F.Cu at (43.0, 170.2)
- added C6: 360pF, Capacitor_SMD:C_0603_1608Metric, F.Cu at (43.0, 160.2)
- added C6: 360pF, Capacitor_SMD:C_0603_1608Metric, F.Cu at (43.0, 150.2)
- added C6: 360pF, Capacitor_SMD:C_0603_1608Metric, F.Cu at (98.5, 129.3)
- added C6: 360pF, Capacitor_SMD:C_0603_1608Metric, F.Cu at (98.5, 139.3)
- added C6: 360pF, Capacitor_SMD:C_0603_1608Metric, F.Cu at (98.5, 169.3)
- added C6: 360pF, Capacitor_SMD:C_0603_1608Metric, F.Cu at (98.5, 159.3)
- added J1: Banana, oscilloscope-probes:SIMPLE_PAD, F.Cu at (64.0, 132.0)
- added J1: Banana, oscilloscope-probes:SIMPLE_PAD, F.Cu at (77.5, 147.5)
- added J1: Banana, oscilloscope-probes:SIMPLE_PAD, F.Cu at (64.0, 162.0)
- added J1: Banana, oscilloscope-probes:SIMPLE_PAD, F.Cu at (64.0, 172.0)
- added J1: Banana, oscilloscope-probes:SIMPLE_PAD, F.Cu at (64.0, 152.0)
- added J1: Banana, oscilloscope-probes:SIMPLE_PAD, F.Cu at (64.0, 142.0)
- added J1: Banana, oscilloscope-probes:SIMPLE_PAD, F.Cu at (77.5, 127.5)
- added J1: Banana, oscilloscope-probes:SIMPLE_PAD, F.Cu at (77.5, 137.5)
- added J1: Banana, oscilloscope-probes:SIMPLE_PAD, F.Cu at (77.5, 167.5)
- added J1: Banana, oscilloscope-probes:SIMPLE_PAD, F.Cu at (77.5, 157.5)
- added J2: Out, oscilloscope-probes:SIMPLE_PAD, B.Cu at (40.1, 169.5)
- added J2: Out, oscilloscope-probes:SIMPLE_PAD, B.Cu at (101.4, 150.0)
- added J2: Out, oscilloscope-probes:SIMPLE_PAD, B.Cu at (40.1, 139.5)
- added J2: Out, oscilloscope-probes:SIMPLE_PAD, B.Cu at (40.1, 129.5)
- added J2: Out, oscilloscope-probes:SIMPLE_PAD, B.Cu at (40.1, 149.5)
- added J2: Out, oscilloscope-probes:SIMPLE_PAD, B.Cu at (40.1, 159.5)
- added J2: Out, oscilloscope-probes:SIMPLE_PAD, B.Cu at (101.4, 130.0)
- added J2: Out, oscilloscope-probes:SIMPLE_PAD, B.Cu at (101.4, 140.0)
- added J2: Out, oscilloscope-probes:SIMPLE_PAD, B.Cu at (101.4, 170.0)
- added J2: Out, oscilloscope-probes:SIMPLE_PAD, B.Cu at (101.4, 160.0)
- added J3: GND, oscilloscope-probes:SIMPLE_PAD, F.Cu at (40.1, 139.5)
- added J3: GND, oscilloscope-probes:SIMPLE_PAD, F.Cu at (101.4, 150.0)
- added J3: GND, oscilloscope-probes:SIMPLE_PAD, F.Cu at (40.1, 129.5)
- added J3: GND, oscilloscope-probes:SIMPLE_PAD, F.Cu at (40.1, 149.5)
- added J3: GND, oscilloscope-probes:SIMPLE_PAD, F.Cu at (40.1, 169.5)
- added J3: GND, oscilloscope-probes:SIMPLE_PAD, F.Cu at (40.1, 159.5)
- added J3: GND, oscilloscope-probes:SIMPLE_PAD, F.Cu at (101.4, 130.0)
- added J3: GND, oscilloscope-probes:SIMPLE_PAD, F.Cu at (101.4, 140.0)
- added J3: GND, oscilloscope-probes:SIMPLE_PAD, F.Cu at (101.4, 170.0)
- added J3: GND, oscilloscope-probes:SIMPLE_PAD, F.Cu at (101.4, 160.0)
- added R1: 10M, oscilloscope-probes:Minimal1206, F.Cu at (59.5, 128.5)
- added R1: 10M, oscilloscope-probes:Minimal1206, F.Cu at (82.0, 151.0)
- added R1: 10M, oscilloscope-probes:Minimal1206, F.Cu at (59.5, 168.5)
- added R1: 10M, oscilloscope-probes:Minimal1206, F.Cu at (59.5, 138.5)
- added R1: 10M, oscilloscope-probes:Minimal1206, F.Cu at (59.5, 148.5)
- added R1: 10M, oscilloscope-probes:Minimal1206, F.Cu at (59.5, 158.5)
- added R1: 10M, oscilloscope-probes:Minimal1206, F.Cu at (82.0, 131.0)
- added R1: 10M, oscilloscope-probes:Minimal1206, F.Cu at (82.0, 141.0)
- added R1: 10M, oscilloscope-probes:Minimal1206, F.Cu at (82.0, 171.0)
- added R1: 10M, oscilloscope-probes:Minimal1206, F.Cu at (82.0, 161.0)
- added R2: 10M, oscilloscope-probes:Minimal1206, F.Cu at (56.1, 128.5)
- added R2: 10M, oscilloscope-probes:Minimal1206, F.Cu at (85.4, 151.0)
- added R2: 10M, oscilloscope-probes:Minimal1206, F.Cu at (56.1, 168.5)
- added R2: 10M, oscilloscope-probes:Minimal1206, F.Cu at (56.1, 138.5)
- added R2: 10M, oscilloscope-probes:Minimal1206, F.Cu at (56.1, 158.5)
- added R2: 10M, oscilloscope-probes:Minimal1206, F.Cu at (56.1, 148.5)
- added R2: 10M, oscilloscope-probes:Minimal1206, F.Cu at (85.4, 131.0)
- added R2: 10M, oscilloscope-probes:Minimal1206, F.Cu at (85.4, 141.0)
- added R2: 10M, oscilloscope-probes:Minimal1206, F.Cu at (85.4, 171.0)
- added R2: 10M, oscilloscope-probes:Minimal1206, F.Cu at (85.4, 161.0)
- added R3: 10M, oscilloscope-probes:Minimal1206, F.Cu at (52.7, 160.7)
- added R3: 10M, oscilloscope-probes:Minimal1206, F.Cu at (88.8, 148.8)
- added R3: 10M, oscilloscope-probes:Minimal1206, F.Cu at (52.7, 140.7)
- added R3: 10M, oscilloscope-probes:Minimal1206, F.Cu at (52.7, 170.7)
- added R3: 10M, oscilloscope-probes:Minimal1206, F.Cu at (52.7, 130.7)
- added R3: 10M, oscilloscope-probes:Minimal1206, F.Cu at (52.7, 150.7)
- added R3: 10M, oscilloscope-probes:Minimal1206, F.Cu at (88.8, 128.8)
- added R3: 10M, oscilloscope-probes:Minimal1206, F.Cu at (88.8, 138.8)
- added R3: 10M, oscilloscope-probes:Minimal1206, F.Cu at (88.8, 168.8)
- added R3: 10M, oscilloscope-probes:Minimal1206, F.Cu at (88.8, 158.8)
- added R4: 10M, oscilloscope-probes:Minimal1206, F.Cu at (49.3, 140.7)
- added R4: 10M, oscilloscope-probes:Minimal1206, F.Cu at (92.2, 148.8)
- added R4: 10M, oscilloscope-probes:Minimal1206, F.Cu at (49.3, 170.7)
- added R4: 10M, oscilloscope-probes:Minimal1206, F.Cu at (49.3, 130.7)
- added R4: 10M, oscilloscope-probes:Minimal1206, F.Cu at (49.3, 160.7)
- added R4: 10M, oscilloscope-probes:Minimal1206, F.Cu at (49.3, 150.7)
- added R4: 10M, oscilloscope-probes:Minimal1206, F.Cu at (92.2, 128.8)
- added R4: 10M, oscilloscope-probes:Minimal1206, F.Cu at (92.2, 138.8)
- added R4: 10M, oscilloscope-probes:Minimal1206, F.Cu at (92.2, 168.8)
- added R4: 10M, oscilloscope-probes:Minimal1206, F.Cu at (92.2, 158.8)
- added R5: 10M, oscilloscope-probes:Minimal1206, F.Cu at (45.9, 130.7)
- added R5: 10M, oscilloscope-probes:Minimal1206, F.Cu at (95.6, 148.8)
- added R5: 10M, oscilloscope-probes:Minimal1206, F.Cu at (45.9, 140.7)
- added R5: 10M, oscilloscope-probes:Minimal1206, F.Cu at (45.9, 170.7)
- added R5: 10M, oscilloscope-probes:Minimal1206, F.Cu at (45.9, 160.7)
- added R5: 10M, oscilloscope-probes:Minimal1206, F.Cu at (45.9, 150.7)
- added R5: 10M, oscilloscope-probes:Minimal1206, F.Cu at (95.6, 128.8)
- added R5: 10M, oscilloscope-probes:Minimal1206, F.Cu at (95.6, 138.8)
- added R5: 10M, oscilloscope-probes:Minimal1206, F.Cu at (95.6, 168.8)
- added R5: 10M, oscilloscope-probes:Minimal1206, F.Cu at (95.6, 158.8)
- added R6: 499k, Resistor_SMD:R_0603_1608Metric, F.Cu at (43.0, 158.8)
- added R6: 499k, Resistor_SMD:R_0603_1608Metric, F.Cu at (98.5, 150.7)
- added R6: 499k, Resistor_SMD:R_0603_1608Metric, F.Cu at (43.0, 128.8)
- added R6: 499k, Resistor_SMD:R_0603_1608Metric, F.Cu at (43.0, 138.8)
- added R6: 499k, Resistor_SMD:R_0603_1608Metric, F.Cu at (43.0, 168.8)
- added R6: 499k, Resistor_SMD:R_0603_1608Metric, F.Cu at (43.0, 148.8)
- added R6: 499k, Resistor_SMD:R_0603_1608Metric, F.Cu at (98.5, 130.7)
- added R6: 499k, Resistor_SMD:R_0603_1608Metric, F.Cu at (98.5, 140.7)
- added R6: 499k, Resistor_SMD:R_0603_1608Metric, F.Cu at (98.5, 170.7)
- added R6: 499k, Resistor_SMD:R_0603_1608Metric, F.Cu at (98.5, 160.7)
- C5: value 10pF 2kV -> 10pF
- moved C5 59.0 mm to (95.6, 151.0)
Routing:
- net Net-(C1-Pad2): track 4.80 -> 120.9 mm, vias 1 -> 20
- net GND: track 1.03 -> 101.8 mm, vias 1 -> 0
- net Net-(C5-Pad1): track 11.0 -> 84.4 mm, vias 1 -> 10
- net Net-(C2-Pad1): track 6.00 -> 50.0 mm
- net Net-(C4-Pad1): track 6.00 -> 50.0 mm
- net Net-(C1-Pad1): track 6.00 -> 50.0 mm
- net Net-(C3-Pad1): track 6.00 -> 50.0 mm
- added copper zone on F.Cu, net Net-(C1-Pad2)
Other:
- board size 19 x 6 mm -> 64.7 x 47.9 mm
- board text added: "Cable to banana, rev 2, 8/2021"
