File: accessories/cable_to_banana/cable_to_banana.sch (KiCad schematic (older format))
At the start: 15 parts, among them J1 Banana, J2 Coax center, J3 Coax shield

Commit message: Revision 4
Parts:
- J2: value Coax center -> Out
- J3: value Coax shield -> GND
